Commit message: Add the laser scan/Problem in Gazebo

File: my_rb1_description/urdf/my_rb1_robot.urdf (robot description, URDF)
Before this commit: robot robot, 5 links, 4 joints
Links:
- added link base_footprint, mass 0.0
- added link link_laser_scan, mass 0.5; collision cylinder length=0.10 radius=0.05; visual cylinder length=0.10 radius=0.05
- link base_link: mass 10 -> 25
Joints:
- added joint joint_base_link: type fixed, parent base_footprint, child base_link, origin xyz=0.0 0.0 0.15 rpy=0 0 0
- added joint joint_laser_scan_chassis: type fixed, parent base_link, child link_laser_scan, origin xyz=0.25 0.0 0.075 rpy=0 0 0

Commit message: Robot Working Good Now

File: my_rb1_description/urdf/my_rb1_robot.urdf (robot description, URDF)
Before this commit: robot robot, 7 links, 6 joints
Links:
- removed link link_back_caster_wheel
- removed link link_front_caster_wheel
- removed link link_laser_scan
- removed link link_left_wheel
- removed link link_right_wheel
- added link back_caster, mass 1; collision sphere radius=0.010; collision sphere radius=0.025
- added link front_caster, mass 1; collision sphere radius=0.010; collision sphere radius=0.025
- added link front_laser, mass 0.5; collision cylinder length=0.10 radius=0.05; visual cylinder length=0.10 radius=0.05
- added link left_wheel, mass 1; collision cylinder length=0.03 radius=0.025; visual cylinder length=0.03 radius=0.025
- added link right_wheel, mass 1; collision cylinder length=0.03 radius=0.025; visual cylinder length=0.03 radius=0.025
Joints:
- joint joint_back_chassis_caster_wheel: child link_back_caster_wheel -> back_caster
- joint joint_chassis_left_wheel: child link_left_wheel -> left_wheel
- joint joint_chassis_right_wheel: child link_right_wheel -> right_wheel
- joint joint_front_chassis_caster_wheel: child link_front_caster_wheel -> front_caster
- joint joint_laser_scan_chassis: child link_laser_scan -> front_laser; origin xyz=0.25 0.0 0.075 rpy=0 0 0 -> xyz=0.25 0.0 0.075 rpy=3.14 0 0

Commit message: Task 2 - Completed

File: my_rb1_description/urdf/my_rb1_robot.urdf (robot description, URDF)
Before this commit: robot robot, 7 links, 6 joints
Links:
- removed link front_laser
Joints:
- removed joint joint_laser_scan_chassis

Commit message: Task 3 - Completed

File: my_rb1_description/urdf/my_rb1_robot.urdf (robot description, URDF)
Before this commit: robot robot, 6 links, 5 joints
Links:
- added link front_laser, mass 0.5; collision cylinder length=0.10 radius=0.05; visual cylinder length=0.10 radius=0.05
Joints:
- added joint joint_laser_scan_chassis: type fixed, parent base_link, child front_laser, origin xyz=0.25 0.0 0.075 rpy=3.14 0 0
